Commit message: Updated urdf file
git-svn-id: https://roboticssrv.wtb.tue.nl/svn/ros/code/tue-ros-pkg/trunk/tue_actuation/amigo_arm_navigation@14634 3a3c2cfb-d3b9-409e-9e75-db8fcdbcaac6

File: urdf/robot_complex.urdf (robot description, URDF)
Before this commit: robot amigo, 128 links, 127 joints
Joints:
- joint back_laser_joint: origin xyz=-0.235 0.0 0.245 rpy=0 0 3.14 -> xyz=-0.27 0.0 0.245 rpy=0 0 3.14

File: urdf/robot_simple.urdf (robot description, URDF)
Before this commit: robot amigo, 80 links, 79 joints
Joints:
- joint back_laser_joint: origin xyz=-0.235 0.0 0.245 rpy=0 0 3.14 -> xyz=-0.27 0.0 0.245 rpy=0 0 3.14

Commit message: Added top laser to Amigo in simulation and changed according arm configuration files
git-svn-id: https://roboticssrv.wtb.tue.nl/svn/ros/code/tue-ros-pkg/trunk/tue_actuation/amigo_arm_navigation@15599 3a3c2cfb-d3b9-409e-9e75-db8fcdbcaac6

File: urdf/robot_complex.urdf (robot description, URDF)
Before this commit: robot amigo, 128 links, 127 joints
Links:
- added link torso_laser, mass 0.5; collision box size=0.05 0.065 0.12; visual box size=0.05 0.065 0.12
- added link torso_lasertop, mass 0.01; collision box size=0.05 0.065 0.01; visual box size=0.05 0.065 0.01
Joints:
- added joint torso_laser_joint: type fixed, parent torso, child torso_laser, origin xyz=-0.08 0.0 0.05 rpy=0 -1.57 0, axis 0 1 0, limit lower=-0.7809 upper=1.5708 effort=13.4 velocity=1.0
- added joint torso_lasertop_joint: type fixed, parent torso_laser, child torso_lasertop
- joint spindle_joint: limit lower=0.0 upper=0.41 effort=30 velocity=1.0 -> lower=0.085 upper=0.41 effort=30 velocity=1.0

File: urdf/robot_simple.urdf (robot description, URDF)
Before this commit: robot amigo, 80 links, 79 joints
Links:
- added link torso_laser, mass 0.5; collision box size=0.05 0.065 0.12; visual box size=0.05 0.065 0.12
- added link torso_lasertop, mass 0.01; collision box size=0.05 0.065 0.01; visual box size=0.05 0.065 0.01
Joints:
- added joint torso_laser_joint: type fixed, parent torso, child torso_laser, origin xyz=-0.08 0.0 0.05 rpy=0 -1.57 0, axis 0 1 0, limit lower=-0.7809 upper=1.5708 effort=13.4 velocity=1.0
- added joint torso_lasertop_joint: type fixed, parent torso_laser, child torso_lasertop
- joint spindle_joint: limit lower=0.0 upper=0.41 effort=30 velocity=1.0 -> lower=0.085 upper=0.41 effort=30 velocity=1.0

Commit message: Updated amigo_arm_navigation/urdf
git-svn-id: https://roboticssrv.wtb.tue.nl/svn/ros/code/tue-ros-pkg/trunk/tue_actuation/amigo_arm_navigation@15932 3a3c2cfb-d3b9-409e-9e75-db8fcdbcaac6

File: urdf/robot_complex.urdf (robot description, URDF)
Before this commit: robot amigo, 130 links, 129 joints
Links:
- removed link hand_marker_left
- removed link hand_marker_right
- removed link omni_sphere10_left_front
- removed link omni_sphere10_left_rear
- removed link omni_sphere10_right_front
- removed link omni_sphere10_right_rear
- removed link omni_sphere11_left_front
- removed link omni_sphere11_left_rear
- removed link omni_sphere11_right_front
- removed link omni_sphere11_right_rear
- removed link omni_sphere12_left_front
- removed link omni_sphere12_left_rear
- removed link omni_sphere12_right_front
- removed link omni_sphere12_right_rear
- removed link omni_sphere1_left_front
- removed link omni_sphere1_left_rear
- removed link omni_sphere1_right_front
- removed link omni_sphere1_right_rear
- removed link omni_sphere2_left_front
- removed link omni_sphere2_left_rear
- removed link omni_sphere2_right_front
- removed link omni_sphere2_right_rear
- removed link omni_sphere3_left_front
- removed link omni_sphere3_left_rear
- removed link omni_sphere3_right_front
- removed link omni_sphere3_right_rear
- removed link omni_sphere4_left_front
- removed link omni_sphere4_left_rear
- removed link omni_sphere4_right_front
- removed link omni_sphere4_right_rear
- removed link omni_sphere5_left_front
- removed link omni_sphere5_left_rear
- removed link omni_sphere5_right_front
- removed link omni_sphere5_right_rear
- removed link omni_sphere6_left_front
- removed link omni_sphere6_left_rear
- removed link omni_sphere6_right_front
- removed link omni_sphere6_right_rear
- removed link omni_sphere7_left_front
- removed link omni_sphere7_left_rear
- removed link omni_sphere7_right_front
- removed link omni_sphere7_right_rear
- removed link omni_sphere8_left_front
- removed link omni_sphere8_left_rear
- removed link omni_sphere8_right_front
- removed link omni_sphere8_right_rear
- removed link omni_sphere9_left_front
- removed link omni_sphere9_left_rear
- removed link omni_sphere9_right_front
- removed link omni_sphere9_right_rear
- removed link wheel_left_front
- removed link wheel_left_rear
- removed link wheel_right_front
- removed link wheel_right_rear
Joints:
- removed joint marker_joint_left
- removed joint marker_joint_right
- removed joint omni_sphere10_joint_left_front
- removed joint omni_sphere10_joint_left_rear
- removed joint omni_sphere10_joint_right_front
- removed joint omni_sphere10_joint_right_rear
- removed joint omni_sphere11_joint_left_front
- removed joint omni_sphere11_joint_left_rear
- removed joint omni_sphere11_joint_right_front
- removed joint omni_sphere11_joint_right_rear
- removed joint omni_sphere12_joint_left_front
- removed joint omni_sphere12_joint_left_rear
- removed joint omni_sphere12_joint_right_front
- removed joint omni_sphere12_joint_right_rear
- removed joint omni_sphere1_joint_left_front
- removed joint omni_sphere1_joint_left_rear
- removed joint omni_sphere1_joint_right_front
- removed joint omni_sphere1_joint_right_rear
- removed joint omni_sphere2_joint_left_front
- removed joint omni_sphere2_joint_left_rear
- removed joint omni_sphere2_joint_right_front
- removed joint omni_sphere2_joint_right_rear
- removed joint omni_sphere3_joint_left_front
- removed joint omni_sphere3_joint_left_rear
- removed joint omni_sphere3_joint_right_front
- removed joint omni_sphere3_joint_right_rear
- removed joint omni_sphere4_joint_left_front
- removed joint omni_sphere4_joint_left_rear
- removed joint omni_sphere4_joint_right_front
- removed joint omni_sphere4_joint_right_rear
- removed joint omni_sphere5_joint_left_front
- removed joint omni_sphere5_joint_left_rear
- removed joint omni_sphere5_joint_right_front
- removed joint omni_sphere5_joint_right_rear
- removed joint omni_sphere6_joint_left_front
- removed joint omni_sphere6_joint_left_rear
- removed joint omni_sphere6_joint_right_front
- removed joint omni_sphere6_joint_right_rear
- removed joint omni_sphere7_joint_left_front
- removed joint omni_sphere7_joint_left_rear
- removed joint omni_sphere7_joint_right_front
- removed joint omni_sphere7_joint_right_rear
- removed joint omni_sphere8_joint_left_front
- removed joint omni_sphere8_joint_left_rear
- removed joint omni_sphere8_joint_right_front
- removed joint omni_sphere8_joint_right_rear
- removed joint omni_sphere9_joint_left_front
- removed joint omni_sphere9_joint_left_rear
- removed joint omni_sphere9_joint_right_front
- removed joint omni_sphere9_joint_right_rear
- removed joint wheel_inner_joint_left_front
- removed joint wheel_inner_joint_left_rear
- removed joint wheel_inner_joint_right_front
- removed joint wheel_inner_joint_right_rear
- joint base_kinect_joint: origin xyz=0.07 0 0.07 rpy=0 0 0 -> xyz=0.07 0 0.07 rpy=0.0 0.01 0.075
- joint spindle_joint: limit lower=0.085 upper=0.41 effort=30 velocity=1.0 -> lower=0.0 upper=0.41 effort=30 velocity=1.0
- joint torso_laser_joint: origin xyz=-0.08 0.0 0.05 rpy=0 -1.57 0 -> xyz=-0.0994 0.0 0.075 rpy=0 -1.57 0

File: urdf/robot_simple.urdf (robot description, URDF)
Before this commit: robot amigo, 82 links, 81 joints
Links:
- removed link base_fixed_link
- removed link base_x_link
- removed link base_y_link
- removed link hand_marker_left
- removed link hand_marker_right
- removed link world
Joints:
- removed joint base_fixed_joint
- removed joint base_phi_joint
- removed joint base_x_joint
- removed joint base_y_joint
- removed joint marker_joint_left
- removed joint marker_joint_right
- joint base_kinect_joint: origin xyz=0.07 0 0.07 rpy=0 0 0 -> xyz=0.07 0 0.07 rpy=0.0 0.01 0.075
- joint spindle_joint: limit lower=0.085 upper=0.41 effort=30 velocity=1.0 -> lower=0.0 upper=0.41 effort=30 velocity=1.0
- joint torso_laser_joint: origin xyz=-0.08 0.0 0.05 rpy=0 -1.57 0 -> xyz=-0.0994 0.0 0.075 rpy=0 -1.57 0
