Commit message: Updated amigo_arm_navigation for tuned torso LRF position
git-svn-id: https://roboticssrv.wtb.tue.nl/svn/ros/code/tue-ros-pkg/trunk/tue_actuation/amigo_arm_navigation@16962 3a3c2cfb-d3b9-409e-9e75-db8fcdbcaac6

File: urdf/robot_complex.urdf (robot description, URDF)
Before this commit: robot amigo, 76 links, 75 joints
Links:
- added link hand_marker_left, mass 1e-05; collision cylinder length=0.0 radius=0.0; visual cylinder length=0.0 radius=0.0
- added link hand_marker_right, mass 1e-05; collision cylinder length=0.0 radius=0.0; visual cylinder length=0.0 radius=0.0
- added link omni_sphere10_left_front, mass 0.05; collision sphere radius=0.03; visual sphere radius=0.03
- added link omni_sphere10_left_rear, mass 0.05; collision sphere radius=0.03; visual sphere radius=0.03
- added link omni_sphere10_right_front, mass 0.05; collision sphere radius=0.03; visual sphere radius=0.03
- added link omni_sphere10_right_rear, mass 0.05; collision sphere radius=0.03; visual sphere radius=0.03
- added link omni_sphere11_left_front, mass 0.05; collision sphere radius=0.03; visual sphere radius=0.03
- added link omni_sphere11_left_rear, mass 0.05; collision sphere radius=0.03; visual sphere radius=0.03
- added link omni_sphere11_right_front, mass 0.05; collision sphere radius=0.03; visual sphere radius=0.03
- added link omni_sphere11_right_rear, mass 0.05; collision sphere radius=0.03; visual sphere radius=0.03
- added link omni_sphere12_left_front, mass 0.05; collision sphere radius=0.03; visual sphere radius=0.03
- added link omni_sphere12_left_rear, mass 0.05; collision sphere radius=0.03; visual sphere radius=0.03
- added link omni_sphere12_right_front, mass 0.05; collision sphere radius=0.03; visual sphere radius=0.03
- added link omni_sphere12_right_rear, mass 0.05; collision sphere radius=0.03; visual sphere radius=0.03
- added link omni_sphere1_left_front, mass 0.05; collision sphere radius=0.03; visual sphere radius=0.03
- added link omni_sphere1_left_rear, mass 0.05; collision sphere radius=0.03; visual sphere radius=0.03
- added link omni_sphere1_right_front, mass 0.05; collision sphere radius=0.03; visual sphere radius=0.03
- added link omni_sphere1_right_rear, mass 0.05; collision sphere radius=0.03; visual sphere radius=0.03
- added link omni_sphere2_left_front, mass 0.05; collision sphere radius=0.03; visual sphere radius=0.03
- added link omni_sphere2_left_rear, mass 0.05; collision sphere radius=0.03; visual sphere radius=0.03
- added link omni_sphere2_right_front, mass 0.05; collision sphere radius=0.03; visual sphere radius=0.03
- added link omni_sphere2_right_rear, mass 0.05; collision sphere radius=0.03; visual sphere radius=0.03
- added link omni_sphere3_left_front, mass 0.05; collision sphere radius=0.03; visual sphere radius=0.03
- added link omni_sphere3_left_rear, mass 0.05; collision sphere radius=0.03; visual sphere radius=0.03
- added link omni_sphere3_right_front, mass 0.05; collision sphere radius=0.03; visual sphere radius=0.03
- added link omni_sphere3_right_rear, mass 0.05; collision sphere radius=0.03; visual sphere radius=0.03
- added link omni_sphere4_left_front, mass 0.05; collision sphere radius=0.03; visual sphere radius=0.03
- added link omni_sphere4_left_rear, mass 0.05; collision sphere radius=0.03; visual sphere radius=0.03
- added link omni_sphere4_right_front, mass 0.05; collision sphere radius=0.03; visual sphere radius=0.03
- added link omni_sphere4_right_rear, mass 0.05; collision sphere radius=0.03; visual sphere radius=0.03
- added link omni_sphere5_left_front, mass 0.05; collision sphere radius=0.03; visual sphere radius=0.03
- added link omni_sphere5_left_rear, mass 0.05; collision sphere radius=0.03; visual sphere radius=0.03
- added link omni_sphere5_right_front, mass 0.05; collision sphere radius=0.03; visual sphere radius=0.03
- added link omni_sphere5_right_rear, mass 0.05; collision sphere radius=0.03; visual sphere radius=0.03
- added link omni_sphere6_left_front, mass 0.05; collision sphere radius=0.03; visual sphere radius=0.03
- added link omni_sphere6_left_rear, mass 0.05; collision sphere radius=0.03; visual sphere radius=0.03
- added link omni_sphere6_right_front, mass 0.05; collision sphere radius=0.03; visual sphere radius=0.03
- added link omni_sphere6_right_rear, mass 0.05; collision sphere radius=0.03; visual sphere radius=0.03
- added link omni_sphere7_left_front, mass 0.05; collision sphere radius=0.03; visual sphere radius=0.03
- added link omni_sphere7_left_rear, mass 0.05; collision sphere radius=0.03; visual sphere radius=0.03
- added link omni_sphere7_right_front, mass 0.05; collision sphere radius=0.03; visual sphere radius=0.03
- added link omni_sphere7_right_rear, mass 0.05; collision sphere radius=0.03; visual sphere radius=0.03
- added link omni_sphere8_left_front, mass 0.05; collision sphere radius=0.03; visual sphere radius=0.03
- added link omni_sphere8_left_rear, mass 0.05; collision sphere radius=0.03; visual sphere radius=0.03
- added link omni_sphere8_right_front, mass 0.05; collision sphere radius=0.03; visual sphere radius=0.03
- added link omni_sphere8_right_rear, mass 0.05; collision sphere radius=0.03; visual sphere radius=0.03
- added link omni_sphere9_left_front, mass 0.05; collision sphere radius=0.03; visual sphere radius=0.03
- added link omni_sphere9_left_rear, mass 0.05; collision sphere radius=0.03; visual sphere radius=0.03
- added link omni_sphere9_right_front, mass 0.05; collision sphere radius=0.03; visual sphere radius=0.03
- added link omni_sphere9_right_rear, mass 0.05; collision sphere radius=0.03; visual sphere radius=0.03
- added link torso_dummy, mass 0; collision cylinder length=0.00 radius=0.0; visual cylinder length=0.00 radius=0.0
- added link wheel_left_front, mass 0.5; collision cylinder length=0.05 radius=0.05; visual cylinder length=0.05 radius=0.05
- added link wheel_left_rear, mass 0.5; collision cylinder length=0.05 radius=0.05; visual cylinder length=0.05 radius=0.05
- added link wheel_right_front, mass 0.5; collision cylinder length=0.05 radius=0.05; visual cylinder length=0.05 radius=0.05
- added link wheel_right_rear, mass 0.5; collision cylinder length=0.05 radius=0.05; visual cylinder length=0.05 radius=0.05
Joints:
- added joint marker_joint_left: type fixed, parent grippoint_left, child hand_marker_left, origin xyz=0.0 0.0 0.0 rpy=0 0 0
- added joint marker_joint_right: type fixed, parent grippoint_right, child hand_marker_right, origin xyz=0.0 0.0 0.0 rpy=0 0 0
- added joint omni_sphere10_joint_left_front: type continuous, parent wheel_left_front, child omni_sphere10_left_front, origin xyz=0.0 0.0 -0.03 rpy=4.7124 0 0, axis 0 1 0, limit effort=0.5 velocity=0.05
- added joint omni_sphere10_joint_left_rear: type continuous, parent wheel_left_rear, child omni_sphere10_left_rear, origin xyz=0.0 0.0 -0.03 rpy=4.7124 0 0, axis 0 1 0, limit effort=0.5 velocity=0.05
- added joint omni_sphere10_joint_right_front: type continuous, parent wheel_right_front, child omni_sphere10_right_front, origin xyz=0.0 0.0 -0.03 rpy=4.7124 0 0, axis 0 1 0, limit effort=0.5 velocity=0.05
- added joint omni_sphere10_joint_right_rear: type continuous, parent wheel_right_rear, child omni_sphere10_right_rear, origin xyz=0.0 0.0 -0.03 rpy=4.7124 0 0, axis 0 1 0, limit effort=0.5 velocity=0.05
- added joint omni_sphere11_joint_left_front: type continuous, parent wheel_left_front, child omni_sphere11_left_front, origin xyz=0.0 0.015 -0.026 rpy=5.236 0 0, axis 0 1 0, limit effort=0.5 velocity=0.05
- added joint omni_sphere11_joint_left_rear: type continuous, parent wheel_left_rear, child omni_sphere11_left_rear, origin xyz=0.0 0.015 -0.026 rpy=5.236 0 0, axis 0 1 0, limit effort=0.5 velocity=0.05
- added joint omni_sphere11_joint_right_front: type continuous, parent wheel_right_front, child omni_sphere11_right_front, origin xyz=0.0 0.015 -0.026 rpy=5.236 0 0, axis 0 1 0, limit effort=0.5 velocity=0.05
- added joint omni_sphere11_joint_right_rear: type continuous, parent wheel_right_rear, child omni_sphere11_right_rear, origin xyz=0.0 0.015 -0.026 rpy=5.236 0 0, axis 0 1 0, limit effort=0.5 velocity=0.05
- added joint omni_sphere12_joint_left_front: type continuous, parent wheel_left_front, child omni_sphere12_left_front, origin xyz=0.0 0.026 -0.015 rpy=5.7596 0 0, axis 0 1 0, limit effort=0.5 velocity=0.05
- added joint omni_sphere12_joint_left_rear: type continuous, parent wheel_left_rear, child omni_sphere12_left_rear, origin xyz=0.0 0.026 -0.015 rpy=5.7596 0 0, axis 0 1 0, limit effort=0.5 velocity=0.05
- added joint omni_sphere12_joint_right_front: type continuous, parent wheel_right_front, child omni_sphere12_right_front, origin xyz=0.0 0.026 -0.015 rpy=5.7596 0 0, axis 0 1 0, limit effort=0.5 velocity=0.05
- added joint omni_sphere12_joint_right_rear: type continuous, parent wheel_right_rear, child omni_sphere12_right_rear, origin xyz=0.0 0.026 -0.015 rpy=5.7596 0 0, axis 0 1 0, limit effort=0.5 velocity=0.05
- added joint omni_sphere1_joint_left_front: type continuous, parent wheel_left_front, child omni_sphere1_left_front, origin xyz=0.0 0.03 0.0 rpy=0.0 0 0, axis 0 1 0, limit effort=0.5 velocity=0.05
- added joint omni_sphere1_joint_left_rear: type continuous, parent wheel_left_rear, child omni_sphere1_left_rear, origin xyz=0.0 0.03 0.0 rpy=0.0 0 0, axis 0 1 0, limit effort=0.5 velocity=0.05
- added joint omni_sphere1_joint_right_front: type continuous, parent wheel_right_front, child omni_sphere1_right_front, origin xyz=0.0 0.03 0.0 rpy=0.0 0 0, axis 0 1 0, limit effort=0.5 velocity=0.05
- added joint omni_sphere1_joint_right_rear: type continuous, parent wheel_right_rear, child omni_sphere1_right_rear, origin xyz=0.0 0.03 0.0 rpy=0.0 0 0, axis 0 1 0, limit effort=0.5 velocity=0.05
- added joint omni_sphere2_joint_left_front: type continuous, parent wheel_left_front, child omni_sphere2_left_front, origin xyz=0.0 0.026 0.015 rpy=0.5236 0 0, axis 0 1 0, limit effort=0.5 velocity=0.05
- added joint omni_sphere2_joint_left_rear: type continuous, parent wheel_left_rear, child omni_sphere2_left_rear, origin xyz=0.0 0.026 0.015 rpy=0.5236 0 0, axis 0 1 0, limit effort=0.5 velocity=0.05
- added joint omni_sphere2_joint_right_front: type continuous, parent wheel_right_front, child omni_sphere2_right_front, origin xyz=0.0 0.026 0.015 rpy=0.5236 0 0, axis 0 1 0, limit effort=0.5 velocity=0.05
- added joint omni_sphere2_joint_right_rear: type continuous, parent wheel_right_rear, child omni_sphere2_right_rear, origin xyz=0.0 0.026 0.015 rpy=0.5236 0 0, axis 0 1 0, limit effort=0.5 velocity=0.05
- added joint omni_sphere3_joint_left_front: type continuous, parent wheel_left_front, child omni_sphere3_left_front, origin xyz=0.0 0.015 0.026 rpy=1.0472 0 0, axis 0 1 0, limit effort=0.5 velocity=0.05
- added joint omni_sphere3_joint_left_rear: type continuous, parent wheel_left_rear, child omni_sphere3_left_rear, origin xyz=0.0 0.015 0.026 rpy=1.0472 0 0, axis 0 1 0, limit effort=0.5 velocity=0.05
- added joint omni_sphere3_joint_right_front: type continuous, parent wheel_right_front, child omni_sphere3_right_front, origin xyz=0.0 0.015 0.026 rpy=1.0472 0 0, axis 0 1 0, limit effort=0.5 velocity=0.05
- added joint omni_sphere3_joint_right_rear: type continuous, parent wheel_right_rear, child omni_sphere3_right_rear, origin xyz=0.0 0.015 0.026 rpy=1.0472 0 0, axis 0 1 0, limit effort=0.5 velocity=0.05
- added joint omni_sphere4_joint_left_front: type continuous, parent wheel_left_front, child omni_sphere4_left_front, origin xyz=0.0 0 0.03 rpy=1.5708 0 0, axis 0 1 0, limit effort=0.5 velocity=0.05
- added joint omni_sphere4_joint_left_rear: type continuous, parent wheel_left_rear, child omni_sphere4_left_rear, origin xyz=0.0 0 0.03 rpy=1.5708 0 0, axis 0 1 0, limit effort=0.5 velocity=0.05
- added joint omni_sphere4_joint_right_front: type continuous, parent wheel_right_front, child omni_sphere4_right_front, origin xyz=0.0 0 0.03 rpy=1.5708 0 0, axis 0 1 0, limit effort=0.5 velocity=0.05
- added joint omni_sphere4_joint_right_rear: type continuous, parent wheel_right_rear, child omni_sphere4_right_rear, origin xyz=0.0 0 0.03 rpy=1.5708 0 0, axis 0 1 0, limit effort=0.5 velocity=0.05
- added joint omni_sphere5_joint_left_front: type continuous, parent wheel_left_front, child omni_sphere5_left_front, origin xyz=0.0 -0.015 0.026 rpy=2.0944 0 0, axis 0 1 0, limit effort=0.5 velocity=0.05
- added joint omni_sphere5_joint_left_rear: type continuous, parent wheel_left_rear, child omni_sphere5_left_rear, origin xyz=0.0 -0.015 0.026 rpy=2.0944 0 0, axis 0 1 0, limit effort=0.5 velocity=0.05
- added joint omni_sphere5_joint_right_front: type continuous, parent wheel_right_front, child omni_sphere5_right_front, origin xyz=0.0 -0.015 0.026 rpy=2.0944 0 0, axis 0 1 0, limit effort=0.5 velocity=0.05
- added joint omni_sphere5_joint_right_rear: type continuous, parent wheel_right_rear, child omni_sphere5_right_rear, origin xyz=0.0 -0.015 0.026 rpy=2.0944 0 0, axis 0 1 0, limit effort=0.5 velocity=0.05
- added joint omni_sphere6_joint_left_front: type continuous, parent wheel_left_front, child omni_sphere6_left_front, origin xyz=0.0 -0.026 0.015 rpy=2.618 0 0, axis 0 1 0, limit effort=0.5 velocity=0.05
- added joint omni_sphere6_joint_left_rear: type continuous, parent wheel_left_rear, child omni_sphere6_left_rear, origin xyz=0.0 -0.026 0.015 rpy=2.618 0 0, axis 0 1 0, limit effort=0.5 velocity=0.05
- added joint omni_sphere6_joint_right_front: type continuous, parent wheel_right_front, child omni_sphere6_right_front, origin xyz=0.0 -0.026 0.015 rpy=2.618 0 0, axis 0 1 0, limit effort=0.5 velocity=0.05
- added joint omni_sphere6_joint_right_rear: type continuous, parent wheel_right_rear, child omni_sphere6_right_rear, origin xyz=0.0 -0.026 0.015 rpy=2.618 0 0, axis 0 1 0, limit effort=0.5 velocity=0.05
- added joint omni_sphere7_joint_left_front: type continuous, parent wheel_left_front, child omni_sphere7_left_front, origin xyz=0.0 -0.03 0.0 rpy=3.1416 0 0, axis 0 1 0, limit effort=0.5 velocity=0.05
- added joint omni_sphere7_joint_left_rear: type continuous, parent wheel_left_rear, child omni_sphere7_left_rear, origin xyz=0.0 -0.03 0.0 rpy=3.1416 0 0, axis 0 1 0, limit effort=0.5 velocity=0.05
- added joint omni_sphere7_joint_right_front: type continuous, parent wheel_right_front, child omni_sphere7_right_front, origin xyz=0.0 -0.03 0.0 rpy=3.1416 0 0, axis 0 1 0, limit effort=0.5 velocity=0.05
- added joint omni_sphere7_joint_right_rear: type continuous, parent wheel_right_rear, child omni_sphere7_right_rear, origin xyz=0.0 -0.03 0.0 rpy=3.1416 0 0, axis 0 1 0, limit effort=0.5 velocity=0.05
- added joint omni_sphere8_joint_left_front: type continuous, parent wheel_left_front, child omni_sphere8_left_front, origin xyz=0.0 -0.026 -0.015 rpy=3.6652 0 0, axis 0 1 0, limit effort=0.5 velocity=0.05
- added joint omni_sphere8_joint_left_rear: type continuous, parent wheel_left_rear, child omni_sphere8_left_rear, origin xyz=0.0 -0.026 -0.015 rpy=3.6652 0 0, axis 0 1 0, limit effort=0.5 velocity=0.05
- added joint omni_sphere8_joint_right_front: type continuous, parent wheel_right_front, child omni_sphere8_right_front, origin xyz=0.0 -0.026 -0.015 rpy=3.6652 0 0, axis 0 1 0, limit effort=0.5 velocity=0.05
- added joint omni_sphere8_joint_right_rear: type continuous, parent wheel_right_rear, child omni_sphere8_right_rear, origin xyz=0.0 -0.026 -0.015 rpy=3.6652 0 0, axis 0 1 0, limit effort=0.5 velocity=0.05
- added joint omni_sphere9_joint_left_front: type continuous, parent wheel_left_front, child omni_sphere9_left_front, origin xyz=0.0 -0.015 -0.026 rpy=4.1888 0 0, axis 0 1 0, limit effort=0.5 velocity=0.05
- added joint omni_sphere9_joint_left_rear: type continuous, parent wheel_left_rear, child omni_sphere9_left_rear, origin xyz=0.0 -0.015 -0.026 rpy=4.1888 0 0, axis 0 1 0, limit effort=0.5 velocity=0.05
- added joint omni_sphere9_joint_right_front: type continuous, parent wheel_right_front, child omni_sphere9_right_front, origin xyz=0.0 -0.015 -0.026 rpy=4.1888 0 0, axis 0 1 0, limit effort=0.5 velocity=0.05
- added joint omni_sphere9_joint_right_rear: type continuous, parent wheel_right_rear, child omni_sphere9_right_rear, origin xyz=0.0 -0.015 -0.026 rpy=4.1888 0 0, axis 0 1 0, limit effort=0.5 velocity=0.05
- added joint torso_dummy_joint: type fixed, parent torso, child torso_dummy, origin xyz=-0.0994 0.0 0.075 rpy=0.0 -1.57 0.0, axis 0 1 0, limit lower=-0.7809 upper=1.5708 effort=13.4 velocity=1.0
- added joint wheel_inner_joint_left_front: type continuous, parent base, child wheel_left_front, origin xyz=-0.2 +0.2 0.005 rpy=0 0 2.3562, axis 1 0 0, limit effort=5.0 velocity=5.0
- added joint wheel_inner_joint_left_rear: type continuous, parent base, child wheel_left_rear, origin xyz=-0.2 -0.2 0.005 rpy=0 0 -2.3562, axis 1 0 0, limit effort=5.0 velocity=5.0
- added joint wheel_inner_joint_right_front: type continuous, parent base, child wheel_right_front, origin xyz=+0.2 +0.2 0.005 rpy=0 0 0.7854, axis 1 0 0, limit effort=5.0 velocity=5.0
- added joint wheel_inner_joint_right_rear: type continuous, parent base, child wheel_right_rear, origin xyz=+0.2 -0.2 0.005 rpy=0 0 -0.7854, axis 1 0 0, limit effort=5.0 velocity=5.0
- joint torso_laser_joint: origin xyz=-0.0994 0.0 0.075 rpy=0 -1.57 0 -> xyz=0.0 0.0 0.0 rpy=0.0 0.0 -0.05; parent torso -> torso_dummy

File: urdf/robot_simple.urdf (robot description, URDF)
Before this commit: robot amigo, 76 links, 75 joints
Links:
- added link base_fixed_link, mass 10
- added link base_x_link, mass 10
- added link base_y_link, mass 10
- added link hand_marker_left, mass 1e-05; collision cylinder length=0.0 radius=0.0; visual cylinder length=0.0 radius=0.0
- added link hand_marker_right, mass 1e-05; collision cylinder length=0.0 radius=0.0; visual cylinder length=0.0 radius=0.0
- added link torso_dummy, mass 0; collision cylinder length=0.00 radius=0.0; visual cylinder length=0.00 radius=0.0
- added link world
Joints:
- added joint base_fixed_joint: type fixed, parent world, child base_fixed_link, origin xyz=0 0 0 rpy=0 0 0
- added joint base_phi_joint: type continuous, parent base_y_link, child base_link, origin xyz=0 0 0 rpy=0 0 0, axis 0 0 1, limit lower=-1000 upper=1000 effort=1000 velocity=1000
- added joint base_x_joint: type prismatic, parent base_fixed_link, child base_x_link, origin xyz=0 0 0 rpy=0 0 0, axis 1 0 0, limit lower=-1000 upper=1000 effort=1000 velocity=1000
- added joint base_y_joint: type prismatic, parent base_x_link, child base_y_link, origin xyz=0 0 0 rpy=0 0 0, axis 0 1 0, limit lower=-1000 upper=1000 effort=1000 velocity=1000
- added joint marker_joint_left: type fixed, parent grippoint_left, child hand_marker_left, origin xyz=0.0 0.0 0.0 rpy=0 0 0
- added joint marker_joint_right: type fixed, parent grippoint_right, child hand_marker_right, origin xyz=0.0 0.0 0.0 rpy=0 0 0
- added joint torso_dummy_joint: type fixed, parent torso, child torso_dummy, origin xyz=-0.0994 0.0 0.075 rpy=0.0 -1.57 0.0, axis 0 1 0, limit lower=-0.7809 upper=1.5708 effort=13.4 velocity=1.0
- joint torso_laser_joint: origin xyz=-0.0994 0.0 0.075 rpy=0 -1.57 0 -> xyz=0.0 0.0 0.0 rpy=0.0 0.0 -0.05; parent torso -> torso_dummy

Commit message: And corresponding arm_navigation_config
git-svn-id: https://roboticssrv.wtb.tue.nl/svn/ros/code/tue-ros-pkg/trunk/tue_actuation/amigo_arm_navigation@17144 3a3c2cfb-d3b9-409e-9e75-db8fcdbcaac6

File: urdf/robot_complex.urdf (robot description, URDF)
Before this commit: robot amigo, 131 links, 130 joints
Joints:
- joint spindle_joint: limit lower=0.0 upper=0.41 effort=30 velocity=1.0 -> lower=0.075 upper=0.41 effort=30 velocity=1.0

File: urdf/robot_simple.urdf (robot description, URDF)
Before this commit: robot amigo, 83 links, 82 joints
Joints:
- joint spindle_joint: limit lower=0.0 upper=0.41 effort=30 velocity=1.0 -> lower=0.075 upper=0.41 effort=30 velocity=1.0

Commit message: new urdf models for changed kinect urdf model
git-svn-id: https://roboticssrv.wtb.tue.nl/svn/ros/code/tue-ros-pkg/trunk/tue_actuation/amigo_arm_navigation@18097 3a3c2cfb-d3b9-409e-9e75-db8fcdbcaac6

File: urdf/robot_complex.urdf (robot description, URDF)
Before this commit: robot amigo, 131 links, 130 joints
Joints:
- joint base_kinect_joint: origin xyz=0.07 0 0.07 rpy=0.0 0.01 0.075 -> xyz=0.07 0.05 0.10 rpy=0 0.01 0.015

File: urdf/robot_simple.urdf (robot description, URDF)
Before this commit: robot amigo, 83 links, 82 joints
Joints:
- joint base_kinect_joint: origin xyz=0.07 0 0.07 rpy=0.0 0.01 0.075 -> xyz=0.07 0.05 0.10 rpy=0 0.01 0.015
