Commit message: Working on conversion to new topic names and message types
git-svn-id: https://roboticssrv.wtb.tue.nl/svn/ros/code/tue-ros-pkg/trunk/tue_actuation/amigo_arm_navigation@18456 3a3c2cfb-d3b9-409e-9e75-db8fcdbcaac6

File: urdf/robot_complex.urdf (robot description, URDF)
Before this commit: robot amigo, 131 links, 130 joints
Links:
- removed link back_laser
- removed link back_lasertop
- removed link base_kinect_openni_camera
- removed link base_kinect_openni_depth_frame
- removed link base_kinect_openni_depth_optical_frame
- removed link base_kinect_openni_rgb_frame
- removed link base_kinect_openni_rgb_optical_frame
- removed link front_laser
- removed link front_lasertop
- removed link hand_marker_left
- removed link hand_marker_right
- removed link omni_sphere10_left_front
- removed link omni_sphere10_left_rear
- removed link omni_sphere10_right_front
- removed link omni_sphere10_right_rear
- removed link omni_sphere11_left_front
- removed link omni_sphere11_left_rear
- removed link omni_sphere11_right_front
- removed link omni_sphere11_right_rear
- removed link omni_sphere12_left_front
- removed link omni_sphere12_left_rear
- removed link omni_sphere12_right_front
- removed link omni_sphere12_right_rear
- removed link omni_sphere1_left_front
- removed link omni_sphere1_left_rear
- removed link omni_sphere1_right_front
- removed link omni_sphere1_right_rear
- removed link omni_sphere2_left_front
- removed link omni_sphere2_left_rear
- removed link omni_sphere2_right_front
- removed link omni_sphere2_right_rear
- removed link omni_sphere3_left_front
- removed link omni_sphere3_left_rear
- removed link omni_sphere3_right_front
- removed link omni_sphere3_right_rear
- removed link omni_sphere4_left_front
- removed link omni_sphere4_left_rear
- removed link omni_sphere4_right_front
- removed link omni_sphere4_right_rear
- removed link omni_sphere5_left_front
- removed link omni_sphere5_left_rear
- removed link omni_sphere5_right_front
- removed link omni_sphere5_right_rear
- removed link omni_sphere6_left_front
- removed link omni_sphere6_left_rear
- removed link omni_sphere6_right_front
- removed link omni_sphere6_right_rear
- removed link omni_sphere7_left_front
- removed link omni_sphere7_left_rear
- removed link omni_sphere7_right_front
- removed link omni_sphere7_right_rear
- removed link omni_sphere8_left_front
- removed link omni_sphere8_left_rear
- removed link omni_sphere8_right_front
- removed link omni_sphere8_right_rear
- removed link omni_sphere9_left_front
- removed link omni_sphere9_left_rear
- removed link omni_sphere9_right_front
- removed link omni_sphere9_right_rear
- removed link openni_camera
- removed link openni_depth_frame
- removed link openni_depth_optical_frame
- removed link openni_rgb_frame
- removed link openni_rgb_optical_frame
- removed link wheel_left_front
- removed link wheel_left_rear
- removed link wheel_right_front
- removed link wheel_right_rear
- added link base_kinect/openni_camera, mass 0.01; collision mesh filename=package://amigo_description/media/meshes/kinect/kinect_with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; visual mesh filename=package://amigo_description/media/meshes/kinect/kinect_with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
- added link base_kinect/openni_depth_frame, mass 0.01
- added link base_kinect/openni_depth_optical_frame, mass 0.001
- added link base_kinect/openni_rgb_frame, mass 0.001
- added link base_kinect/openni_rgb_optical_frame, mass 0.001
- added link base_laser, mass 0.5; collision box size=0.05 0.065 0.12; visual box size=0.05 0.065 0.12
- added link lasertop, mass 0.01; collision box size=0.05 0.065 0.01; visual box size=0.05 0.065 0.01
- added link top_kinect/openni_camera, mass 0.01; visual box size=0 0 0
- added link top_kinect/openni_depth_frame, mass 0.01
- added link top_kinect/openni_depth_optical_frame, mass 0.001
- added link top_kinect/openni_rgb_frame, mass 0.001
- added link top_kinect/openni_rgb_optical_frame, mass 0.001
- link base: geometry collision mesh filename=package://amigo_description/media/meshes/bottomcovers.dae scale=0.0004 0.0004 0.0004; visual mesh filename=package://amigo_description/media/meshes/bottomcovers.dae scale=0.0004 0.0004 0.0004
- link finger1_left: mass 0.05 -> 0.01
- link finger1_right: mass 0.05 -> 0.01
- link finger1_tip_left: mass 0.05 -> 0.01
- link finger1_tip_right: mass 0.05 -> 0.01
- link finger2_left: mass 0.05 -> 0.01
- link finger2_right: mass 0.05 -> 0.01
- link finger2_tip_left: mass 0.05 -> 0.01
- link finger2_tip_right: mass 0.05 -> 0.01
- link fore_arm_left: mass 0.1 -> 0.85; geometry collision mesh filename=package://amigo_description/media/meshes/forearmtextured.dae scale=0.0004 0.0004 0.0004; visual mesh filename=package://amigo_description/media/meshes/forearmtextured.dae scale=0.0004 0.0004 0.0004
- link fore_arm_right: mass 0.1 -> 0.85; geometry collision mesh filename=package://amigo_description/media/meshes/forearmtextured.dae scale=0.0004 0.0004 0.0004; visual mesh filename=package://amigo_description/media/meshes/forearmtextured.dae scale=0.0004 0.0004 0.0004
- link head: geometry collision mesh filename=package://amigo_description/media/meshes/headtextured.dae scale=0.0004 0.0004 0.0004; visual mesh filename=package://amigo_description/media/meshes/headtextured.dae scale=0.0004 0.0004 0.0004
- link logo: geometry collision mesh filename=package://amigo_description/media/meshes/logo.dae scale=0.0016 0.0016 0.0016; visual mesh filename=package://amigo_description/media/meshes/logo.dae scale=0.0016 0.0016 0.0016
- link neck_tilt: geometry collision mesh filename=package://amigo_description/media/meshes/necktilttextured.d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 scale=0.004 0.004 0.004; visual mesh filename=package://amigo_description/media/meshes/necktilttextured.d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 scale=0.004 0.004 0.004
- link shoulder_link1_left: mass 0.1 -> 0.25
- link shoulder_link1_right: mass 0.1 -> 0.25
- link shoulder_link2_left: mass 0.1 -> 0.15
- link shoulder_link2_right: mass 0.1 -> 0.15
- link shoulder_mount_left: mass 0.1 -> 0.15
- link shoulder_mount_right: mass 0.1 -> 0.15
- link torso: geometry collision mesh filename=package://amigo_description/media/meshes/torsocovers.dae scale=0.0004 0.0004 0.0004; visual mesh filename=package://amigo_description/media/meshes/torsocovers.dae scale=0.0004 0.0004 0.0004
- link torso_assist_slider_back: geometry collision mesh filename=package://amigo_description/media/meshes/torsoassistslidert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 scale=0.004 0.004 0.005; visual mesh filename=package://amigo_description/media/meshes/torsoassistslidert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 scale=0.004 0.004 0.005
- link torso_assist_slider_left: geometry collision mesh filename=package://amigo_description/media/meshes/torsoassistslidert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 scale=0.004 0.004 0.005; visual mesh filename=package://amigo_description/media/meshes/torsoassistslidert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 scale=0.004 0.004 0.005
- link torso_assist_slider_right: geometry collision mesh filename=package://amigo_description/media/meshes/torsoassistslidert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 scale=0.004 0.004 0.005; visual mesh filename=package://amigo_description/media/meshes/torsoassistslidert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 scale=0.004 0.004 0.005
- link torso_slider: geometry collision mesh filename=package://amigo_description/media/meshes/torsoslidertexture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 scale=0.004 0.004 0.004; visual mesh filename=package://amigo_description/media/meshes/torsoslidertexture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 scale=0.004 0.004 0.004
- link upper_arm_left: mass 2.9 -> 2.95; geometry collision mesh filename=package://amigo_description/media/meshes/upperarmtextured.d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 scale=0.0004 0.0004 0.0004; visual mesh filename=package://amigo_description/media/meshes/upperarmtextured.d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 scale=0.0004 0.0004 0.0004
- link upper_arm_right: mass 2.9 -> 2.95; geometry collision mesh filename=package://amigo_description/media/meshes/upperarmtextured.d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 scale=0.0004 0.0004 0.0004; visual mesh filename=package://amigo_description/media/meshes/upperarmtextured.d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 scale=0.0004 0.0004 0.0004
Joints:
- removed joint back_laser_joint
- removed joint back_lasertop_joint
- removed joint base_kinect_base_kinect_joint
- removed joint base_kinect_joint
- removed joint base_kinect_kinect_depth_joint
- removed joint base_kinect_kinect_depth_optical_joint
- removed joint base_kinect_kinect_rgb_joint
- removed joint base_kinect_kinect_rgb_optical_joint
- removed joint front_laser_joint
- removed joint front_lasertop_joint
- removed joint kinect_depth_joint
- removed joint kinect_depth_optical_joint
- removed joint kinect_rgb_joint
- removed joint kinect_rgb_optical_joint
- removed joint marker_joint_left
- removed joint marker_joint_right
- removed joint omni_sphere10_joint_left_front
- removed joint omni_sphere10_joint_left_rear
- removed joint omni_sphere10_joint_right_front
- removed joint omni_sphere10_joint_right_rear
- removed joint omni_sphere11_joint_left_front
- removed joint omni_sphere11_joint_left_rear
- removed joint omni_sphere11_joint_right_front
- removed joint omni_sphere11_joint_right_rear
- removed joint omni_sphere12_joint_left_front
- removed joint omni_sphere12_joint_left_rear
- removed joint omni_sphere12_joint_right_front
- removed joint omni_sphere12_joint_right_rear
- removed joint omni_sphere1_joint_left_front
- removed joint omni_sphere1_joint_left_rear
- removed joint omni_sphere1_joint_right_front
- removed joint omni_sphere1_joint_right_rear
- removed joint omni_sphere2_joint_left_front
- removed joint omni_sphere2_joint_left_rear
- removed joint omni_sphere2_joint_right_front
- removed joint omni_sphere2_joint_right_rear
- removed joint omni_sphere3_joint_left_front
- removed joint omni_sphere3_joint_left_rear
- removed joint omni_sphere3_joint_right_front
- removed joint omni_sphere3_joint_right_rear
- removed joint omni_sphere4_joint_left_front
- removed joint omni_sphere4_joint_left_rear
- removed joint omni_sphere4_joint_right_front
- removed joint omni_sphere4_joint_right_rear
- removed joint omni_sphere5_joint_left_front
- removed joint omni_sphere5_joint_left_rear
- removed joint omni_sphere5_joint_right_front
- removed joint omni_sphere5_joint_right_rear
- removed joint omni_sphere6_joint_left_front
- removed joint omni_sphere6_joint_left_rear
- removed joint omni_sphere6_joint_right_front
- removed joint omni_sphere6_joint_right_rear
- removed joint omni_sphere7_joint_left_front
- removed joint omni_sphere7_joint_left_rear
- removed joint omni_sphere7_joint_right_front
- removed joint omni_sphere7_joint_right_rear
- removed joint omni_sphere8_joint_left_front
- removed joint omni_sphere8_joint_left_rear
- removed joint omni_sphere8_joint_right_front
- removed joint omni_sphere8_joint_right_rear
- removed joint omni_sphere9_joint_left_front
- removed joint omni_sphere9_joint_left_rear
- removed joint omni_sphere9_joint_right_front
- removed joint omni_sphere9_joint_right_rear
- removed joint spindle_joint
- removed joint wheel_inner_joint_left_front
- removed joint wheel_inner_joint_left_rear
- removed joint wheel_inner_joint_right_front
- removed joint wheel_inner_joint_right_rear
- added joint base_kinect/base_kinect_joint: type fixed, parent base, child base_kinect/openni_camera, origin xyz=0.3 0 0.26 rpy=0 -0.07 0
- added joint base_kinect/kinect_depth_joint: type fixed, parent base_kinect/openni_camera, child base_kinect/openni_depth_frame, origin xyz=0 0.018 0 rpy=0 0 0
- added joint base_kinect/kinect_depth_optical_joint: type fixed, parent base_kinect/openni_depth_frame, child base_kinect/openni_depth_optical_frame, origin xyz=0 0 0 rpy=-1.570795 0 -1.570795
- added joint base_kinect/kinect_rgb_joint: type fixed, parent base_kinect/openni_camera, child base_kinect/openni_rgb_frame, origin xyz=0 -0.005 0 rpy=0 0 0
- added joint base_kinect/kinect_rgb_optical_joint: type fixed, parent base_kinect/openni_rgb_frame, child base_kinect/openni_rgb_optical_frame, origin xyz=0 0 0 rpy=-1.570795 0 -1.570795
- added joint base_laser_joint: type fixed, parent base, child base_laser, origin xyz=0.31 0.0 0.185 rpy=0 0 0, axis 0 1 0, limit lower=-0.7809 upper=1.5708 effort=13.4 velocity=1.0
- added joint lasertop_joint: type fixed, parent base_laser, child lasertop
- added joint top_kinect/base_kinect_joint: type fixed, parent head, child top_kinect/openni_camera, origin xyz=0.07 0 0.07 rpy=0 0 0
- added joint top_kinect/kinect_depth_joint: type fixed, parent top_kinect/openni_camera, child top_kinect/openni_depth_frame, origin xyz=0 0.018 0 rpy=0 0 0
- added joint top_kinect/kinect_depth_optical_joint: type fixed, parent top_kinect/openni_depth_frame, child top_kinect/openni_depth_optical_frame, origin xyz=0 0 0 rpy=-1.570795 0 -1.570795
- added joint top_kinect/kinect_rgb_joint: type fixed, parent top_kinect/openni_camera, child top_kinect/openni_rgb_frame, origin xyz=0 -0.005 0 rpy=0 0 0
- added joint top_kinect/kinect_rgb_optical_joint: type fixed, parent top_kinect/openni_rgb_frame, child top_kinect/openni_rgb_optical_frame, origin xyz=0 0 0 rpy=-1.570795 0 -1.570795
- added joint torso_joint: type prismatic, parent base, child torso_slider, origin xyz=0.0 0.0 0.58 rpy=3.14159265 -1.5708 0, axis 1 0 0, limit lower=0.0 upper=0.41 effort=1000 velocity=10.0
- joint finger1_joint_left: limit lower=-1.57 upper=1.57 effort=3 velocity=1.0 -> lower=0.2 upper=1 effort=3 velocity=1.0
- joint finger1_joint_right: limit lower=-1.57 upper=1.57 effort=3 velocity=1.0 -> lower=0.2 upper=1 effort=3 velocity=1.0
- joint finger1_tip_joint_left: limit lower=-1.57 upper=1.57 effort=3 velocity=1.0 -> lower=-0.6 upper=-0.2 effort=3 velocity=1.0
- joint finger1_tip_joint_right: limit lower=-1.57 upper=1.57 effort=3 velocity=1.0 -> lower=-0.6 upper=-0.2 effort=3 velocity=1.0
- joint finger2_joint_left: limit lower=-1.57 upper=1.57 effort=3 velocity=1.0 -> lower=0.2 upper=1 effort=3 velocity=1.0
- joint finger2_joint_right: limit lower=-1.57 upper=1.57 effort=3 velocity=1.0 -> lower=0.2 upper=1 effort=3 velocity=1.0
- joint finger2_tip_joint_left: limit lower=-1.57 upper=1.57 effort=3 velocity=1.0 -> lower=-0.6 upper=-0.2 effort=3 velocity=1.0
- joint finger2_tip_joint_right: limit lower=-1.57 upper=1.57 effort=3 velocity=1.0 -> lower=-0.6 upper=-0.2 effort=3 velocity=1.0
- joint logo_joint: parent front_laser -> base_laser
