Commit message: Removed complex and simple model and added amigo.urdf to be able to check differences on Jenkins
git-svn-id: https://roboticssrv.wtb.tue.nl/svn/ros/code/tue-ros-pkg/trunk/tue_actuation/amigo_arm_navigation@18910 3a3c2cfb-d3b9-409e-9e75-db8fcdbcaac6

File: urdf/amigo.urdf (robot description, URDF)
Before this commit: robot amigo, 75 links, 74 joints
Joints:
- joint neck_tilt_joint: limit lower=-2.0 upper=2.0 effort=13.4 velocity=1.0 -> lower=-0.5 upper=0.88 effort=13.4 velocity=1.0
